File: KicadJE-EuroPowerSupply2-PCB.kicad_pcb (KiCad board)
At the start: 2 copper layers, 159 x 128 mm, 143 parts, among them J101 Laptop Power, J102 +-15V thru, J103 +-12v out, J104 +5V out, J105 Laptop Power Out, J106 FrontInterConnVin, J107 FrontInterConnVin, J108 Conn_01x08, J109 Conn_01x08, P101 Doepfer_Power_10pin, P102 Doepfer_Power_16pin, P105 Doepfer_Power_10pin, P106 Doepfer_Power_16pin, Q201 TIP41, Q202 TIP41, Q203 TIP42, Q204 MMBT2907A, Q205 MMBT2222A, Q206 MMBT2907A, SW101 SW_SPDT, U201 LM7812_TO220, U202 LM7805_TO220, U203 Step Down Module +15 to 7v - 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, U204 LM7912_TO220, U205 XL6009 Module DCDC 19 to 30v, U206 TL071, U207 LM78M05_TO252, U208 LM78M12_TO252, U209 MC79M12_TO252

Commit message: PCB Gerber
Gerber
Parts:
- removed H101, H102: MountingHole_Pad, AJ:MountingHole_Eurorack3
- removed H105 (x3): OL, AJ:LED_Hole_3mm
- removed H105 (x4): ON, AJ:LED_Hole_3mm
- removed TP109: Tri, AJ:Jack_6m3
- removed TP110 (x2): SQ, AJ:Jack_6m3
- moved G*** 124.5 mm to (125.0, 145.0)
Other:
- board size 159 x 128 mm -> 100 x 100 mm
- board text removed: "+12"
- board text removed: "+5"
- board text removed: "-12"
- board text removed: "In"
- board text removed: "Out"
- board text removed: "on"
