File: KicadJE-EuroPowerSupply2-Faceplate.kicad_pcb (KiCad board)
At the start: 2 copper layers, 20 x 128 mm, 13 parts

Commit message: Gerber update
Other:
- board text added: "JLCJLCJLCJLC"
Changed lines of the file:
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@@
   (general
     (thickness 1.6)
-    (drawings 72)
+    (drawings 73)
     (tracks 0)
     (zones 0)
@@
     (pad "" np_thru_hole circle (at 0 0) (size 3 3) (drill 3) (layers *.Cu *.Mask))
   )
+  (gr_text JLCJLCJLCJLC (at 10.5 163) (layer B.SilkS)
+    (effects (font (size 0.9 0.9) (thickness 0.2)) (justify left mirror))
+  )
   (gr_text "Johansen Engineering\nPWR2 - Rev A\n15/03-2020" (at 9.5 95) (layer B.SilkS)
